File: hardware/dya-dash/left/dya-left.kicad_sch (KiCad schematic)
At the start: 113 parts

Commit message: Finalize v2
Parts:
- added QL8: Q_PMOS_GSD, Package_TO_SOT_SMD:SOT-23, symbol Device:Q_PMOS_GSD
- added RL13: 100kΩ, Resistor_SMD:R_0805_2012Metric, symbol Device:R
- RL15: value 1kΩ -> 100Ω; LCSC C17513 -> C17408
- SWL24, SWL25: footprint Button_Switch_THT:SW_PUSH_1P1T_6x3.5mm_H4.3_APEM_MJTP1243 -> 0_dya-kbd:Push_PTS636SM43SMTR
- SW_BATL1: footprint 0_kbd_Parts:TGSW_MSK-12D19 -> 0_dya-kbd:MK-12C02-G015; LCSC (none) -> C2890358
Connections:
- net GNDL: now also RL13.1
- net at SW_BATL1.1 (A): now also JL4.2 (Pin_2)
- net at SW_BATL1.3 (C): no longer JL4.2 (Pin_2)
- net at CL5.1, LL1.1, RL2.1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: now also QL8.2 (S); no longer JL4.1 (Pin_1)
- new net: QL8.1 (G), RL13.2
- new net: JL4.1 (Pin_1), QL8.3 (D)
Other:
- note added: "1.0V reset"
- note added: "Backflow prevention from USB power"
- note added: "Low VGS(th) required"
- note added: "Reverse connection protection"
- note removed: "Backflow prevention"
- moved on the sheet: JL4, RL2, RL3, SW_BATL1
