File: hardware/dya-dash/panelized/dya-panelized.kicad_sch (KiCad schematic)
At the start: 250 parts, among them J1 Conn_01x06_Pin, U1 PMW3610, U2 TLV70018_SOT23-5

Commit message: Finalize v2
Parts:
- removed CR5, CR7: 10uF, Capacitor_SMD:C_0805_2012Metric, symbol Device:C
- removed DL10, DL11, DL23, DL24, DL27, DL28, DL30, DL33, DL39, DR13, DR14, DR25, DR26, DR3, DR31, DR32, DR35, DR37, DR42, DR6: D, Diode_SMD:D_SOD-123, symbol Device:D
- removed JL3: Conn_01x04, 0_dya-kbd:JUSHUO-AFH34-S06FIA-1H, symbol Connector_Generic:Conn_01x06
- removed JL4: Conn_01x02_Pin, 0_dya-kbd:AAA-battery, symbol Connector:Conn_01x02_Pin
- removed JR1: USB_C_Receptacle_USB2.0_14P, Connector_USB:USB_C_Receptacle_G-Switch_GT-USB-7010ASV, symbol Connector:USB_C_Receptacle_USB2.0_14P
- removed QR6: Q_PMOS_GSD, Package_TO_SOT_SMD:SOT-23, symbol Device:Q_PMOS_GSD
- removed RL1, RL4, RR12: 100kΩ, Resistor_SMD:R_0805_2012Metric, symbol Device:R
- removed RL10, RL11: 100Ω, Resistor_SMD:R_0805_2012Metric, symbol Device:R
- removed RR15: 1kΩ, Resistor_SMD:R_0805_2012Metric, symbol Device:R
- removed RR2: 1MΩ, Resistor_SMD:R_0805_2012Metric, symbol Device:R
- removed RR6: 470kΩ, Resistor_SMD:R_0805_2012Metric, symbol Device:R
- removed RR7: 150kΩ, Resistor_SMD:R_0805_2012Metric, symbol Device:R
- removed SWL1, SWL12, SWL15, SWL3, SWR10, SWR13, SWR14, SWR18, SWR2, SWR22, SWR5, SWR6: SW_Push_45deg, 0_dya-kbd:Kailh-PG1353-Hotswap-1U, symbol Switch:SW_Push_45deg
- removed SWL24, SWL25: SW_Push_45deg, Button_Switch_THT:SW_PUSH_1P1T_6x3.5mm_H4.3_APEM_MJTP1243, symbol Switch:SW_Push_45deg
- removed SWR19: SW_Push_45deg, 0_dya-kbd:Soft-sw-push-C4817, symbol Switch:SW_Push_45deg
- removed UL4: TTP224, Package_SO:SSOP-16_3.9x4.9mm_P0.635mm, symbol 0_dya-kbd:TTP224
- removed UR3: BU42, 0_dya-kbd:BU42XX, symbol 0_dya-kbd:BU42
- added CL5, CL7: 10uF, Capacitor_SMD:C_0805_2012Metric, symbol Device:C
- added DL13, DL14, DL25, DL26, DL3, DL31, DL32, DL35, DL37, DL42, DL6, DR10, DR11, DR23, DR24, DR27, DR28, DR30, DR33, DR39, DR43, DR44, DR45, DR46: D, Diode_SMD:D_SOD-123, symbol Device:D
- added JL1: USB_C_Receptacle_USB2.0_14P, Connector_USB:USB_C_Receptacle_G-Switch_GT-USB-7010ASV, symbol Connector:USB_C_Receptacle_USB2.0_14P
- added JR3: Conn_01x04, 0_dya-kbd:JUSHUO-AFH34-S06FIA-1H, symbol Connector_Generic:Conn_01x06
- added JR4: Conn_01x02_Pin, 0_dya-kbd:AAA-battery, symbol Connector:Conn_01x02_Pin
- added QL6, QL8, QR8: Q_PMOS_GSD, Package_TO_SOT_SMD:SOT-23, symbol Device:Q_PMOS_GSD
- added RL12, RL13, RR1, RR13, RR4: 100kΩ, Resistor_SMD:R_0805_2012Metric, symbol Device:R
- added RL15, RR10, RR11: 100Ω, Resistor_SMD:R_0805_2012Metric, symbol Device:R
- added RL2: 1MΩ, Resistor_SMD:R_0805_2012Metric, symbol Device:R
- added RL6: 470kΩ, Resistor_SMD:R_0805_2012Metric, symbol Device:R
- added RL7: 150kΩ, Resistor_SMD:R_0805_2012Metric, symbol Device:R
- added SWL10, SWL13, SWL14, SWL18, SWL19, SWL2, SWL22, SWL5, SWL6, SWR1, SWR12, SWR15, SWR3: SW_Push_45deg, 0_dya-kbd:Kailh-PG1353-Hotswap-1U, symbol Switch:SW_Push_45deg
- added SWR24, SWR25: SW_Push_45deg, 0_dya-kbd:Soft-sw-push-C4817, symbol Switch:SW_Push_45deg
- added SWR27, SWR28: SW_Push_45deg, 0_dya-kbd:Push_PTS636SM43SMTR, symbol Switch:SW_Push_45deg
- added UL3: BU42, 0_dya-kbd:BU42XX, symbol 0_dya-kbd:BU42
- added UR4: TTP224, Package_SO:SSOP-16_3.9x4.9mm_P0.635mm, symbol 0_dya-kbd:TTP224
- RR15: renamed from RL15; value 1kΩ -> 100Ω; LCSC C17513 -> C17408
- SWL24: renamed from SWR24; footprint 0_dya-kbd:Soft-sw-push-C4817 -> 0_dya-kbd:Push_PTS636SM43SMTR
- SWL25: renamed from SWR25; footprint 0_dya-kbd:Soft-sw-push-C4817 -> 0_dya-kbd:Push_PTS636SM43SMTR
- SWR19: renamed from SWL19; footprint 0_dya-kbd:Kailh-PG1353-Hotswap-1U -> 0_dya-kbd:Soft-sw-push-C4817; LCSC C5333465 -> (none)
- SW_BATL1, SW_BATR1: footprint 0_kbd_Parts:TGSW_MSK-12D19 -> 0_dya-kbd:MK-12C02-G015; LCSC (none) -> C963206
- renumbered CL5 to CR5, CL7 to CR7, DR10 to DL10, DR11 to DL11, DR23 to DL23, DR24 to DL24, DR27 to DL27, DR28 to DL28, DR30 to DL30, DR33 to DL33, DR39 to DL39, DL13 to DR13, DL14 to DR14, DL25 to DR25, DL26 to DR26, DL3 to DR3, DL31 to DR31, DL32 to DR32, DL35 to DR35, DL37 to DR37, DL42 to DR42, DL6 to DR6, JR3 to JL3, JR4 to JL4, JL1 to JR1, QL6 to QR6, RR1 to RL1, RR10 to RL10, RR11 to RL11, RR4 to RL4, RL12 to RR12, RL2 to RR2, RL6 to RR6, RL7 to RR7, SWR1 to SWL1, SWR12 to SWL12, SWR15 to SWL15, SWR3 to SWL3, SWL10 to SWR10, SWL13 to SWR13, SWL14 to SWR14, SWL18 to SWR18, SWL2 to SWR2, SWL22 to SWR22, SWL5 to SWR5, SWL6 to SWR6, UR4 to UL4, UL3 to UR3
Connections:
- net 3.3V_L: now also JL3.1 (Pin_1), UL4.5 (AHLB), UL4.6 (VDD)
- net 3.3V_R: now also JR3.1 (Pin_1), UR4.5 (AHLB), UR4.6 (VDD); no longer JL3.1 (Pin_1), UL4.5 (AHLB), UL4.6 (VDD)
- net BAT_L: now also QL6.2 (S); no longer QR6.2 (S)
- net BAT_R: now also QR6.2 (S)
- net GNDL: now also CL5.2, CL7.2, JL1.A1 (GND), JL1.A12 (GND), JL1.B1 (GND), JL1.B12 (GND), JL1.S1 (SHIELD), JR3.5 (Pin_5), RL12.2, RL13.1, RL7.2, RR1.1, RR13.2, UL3.3 (GND), UR4.10 (VSS)
- net INPUT_VOLTAGE_L: now also RL2.2; no longer RR2.2
- net INPUT_VOLTAGE_R: now also RR2.2
- net LR_COM: now also JL1.A6 (D+), JL1.B6 (D+), RL15.1; no longer JR1.A6 (D+), JR1.B6 (D+), RR15.1
- net LR_COM_R: now also JR1.A6 (D+), JR1.B6 (D+), RR15.1
- net MOTION_L: now also JL3.4 (Pin_4)
- net MOTION_OR_LR_COM_L: now also RL15.2; no longer RR15.2
- net MOTION_OR_LR_COM_R: now also RR15.2
- net MOTION_R: now also JR3.4 (Pin_4); no longer JL3.4 (Pin_4)
- net PINL0: now also DL3.1 (K), DL6.1 (K); no longer DR3.1 (K), DR6.1 (K)
- net PINL1: now also DL10.2 (A), DL11.2 (A)
- net PINL2: now also DL13.2 (A), DL14.1 (K); no longer DR13.2 (A), DR14.1 (K)
- net PINL3: now also DL23.2 (A)
- net PINL4: now also DL27.2 (A), DL28.1 (K), DL25.2 (A), DL26.2 (A); no longer DR25.2 (A), DR26.2 (A)
- net PINL5: now also DL33.2 (A), DL31.2 (A), DL32.2 (A), DL35.1 (K); no longer DR31.2 (A), DR32.2 (A), DR35.1 (K)
- net PINL6: now also DL39.2 (A), DL37.2 (A), DL42.1 (K); no longer DR37.2 (A), DR42.1 (K)
- net PINR0: now also DR3.1 (K), DR6.1 (K)
- net PINR1: now also DR10.2 (A), DR11.2 (A); no longer DL10.2 (A), DL11.2 (A)
- net PINR2: now also DR13.2 (A), DR14.1 (K)
- net PINR3: now also DR23.2 (A); no longer DL23.2 (A)
- net PINR4: now also DR25.2 (A), DR26.2 (A), DR27.2 (A), DR28.1 (K); no longer DL27.2 (A), DL28.1 (K)
- net PINR5: now also DR31.2 (A), DR32.2 (A), DR35.1 (K), DR33.2 (A); no longer DL33.2 (A)
- net PINR6: now also DR37.2 (A), DR42.1 (K), DR39.2 (A), SWR27.2, SWR28.2; no longer DL39.2 (A)
- net SCLK_L: now also JL3.2 (Pin_2)
- net SCLK_R: now also JR3.2 (Pin_2); no longer JL3.2 (Pin_2)
- net SDIO_L: now also JL3.3 (Pin_3)
- net SDIO_R: now also JR3.3 (Pin_3); no longer JL3.3 (Pin_3)
- net TOUCHL3: now also RL10.1
- net TOUCHL4: now also RL11.1
- net TOUCHR3: now also RR10.1; no longer RL10.1
- net TOUCHR4: now also RR11.1; no longer RL11.1
- net VBUS_L: now also JL1.A4 (VBUS), JL1.A9 (VBUS), JL1.B4 (VBUS), JL1.B9 (VBUS), QL6.1 (G), RL12.1; no longer JR1.A4 (VBUS), JR1.A9 (VBUS), JR1.B4 (VBUS), JR1.B9 (VBUS), QR6.1 (G), RR12.1
- net VBUS_R: now also JR1.A4 (VBUS), JR1.A9 (VBUS), JR1.B4 (VBUS), JR1.B9 (VBUS), QR6.1 (G), RR12.1
- net at DL2.2 (A), SWL11.1, SWL23.1: now also SWL1.1, SWL15.1, DL14.2 (A), SWL19.1; no longer DR14.2 (A), SWR19.1
- net at CL2.1, TL2.1 (Pin_1): now also UL4.2 (TP1)
- net at SW_BATL1.1 (A): now also JL4.2 (Pin_2)
- net at CR5.1, RR2.1, UR3.2 (VDD): now also LR1.1, UR2.8 (VIN), QR8.2 (S), RR4.2; no longer LL1.1, UL2.8 (VIN)
- net at DL27.1 (K): now also SWL16.2; no longer SWR16.2
- net at CR3.1, TR3.1 (Pin_1): now also UR4.3 (TP2); no longer UL4.3 (TP2)
- net at CL1.1, TL1.1 (Pin_1): now also UL4.1 (TP0)
- net at CL4.1, TL4.1 (Pin_1): now also UL4.4 (TP3)
- net at DL21.2 (A), SWL16.1, SWL20.1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: now also SWL24.1, DL3.2 (A), SWL2.1; no longer DR3.2 (A), SWR2.1
- net at DL40.1 (K): now also SWL25.2
- net at DR1.2 (A), DR7.2 (A): now also SWR10.1, SWR14.1, SWR18.1, SWR22.1, SWR6.1
- net at DR19.1 (K): now also SWR10.2
- net at UR3.1 (Vout): now also UR2.5 (EN), RR4.1; no longer UL2.5 (EN)
- net at SWR2.2: now also DR9.1 (K); no longer DL9.1 (K)
- net LABEL_CR5: now reaches DR5.2 (A), SWR17.1, SWR26.1, SWR4.1, SWR9.1
- net LABEL_CR5: now also DR35.2 (A), SWR13.1, DR46.1 (K)
- net at DL23.1 (K): now also SWL13.2
- net at JPL1.1 (A): now also UL4.8 (LPMB)
- net at SWL20.2: now also DL33.1 (K)
- net at DL28.2 (A), SWL12.1, SWL25.1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: now also DL4.2 (A), SWL21.1, SWL8.1; no longer DR4.2 (A), SWR21.1, SWR8.1
- net at CL6.1, CL8.1, UL2.3 (VOUT)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: now also CL7.1, QL6.3 (D), RL6.1; no longer CR7.1, QR6.3 (D), RR6.1
- net LABEL_CR3: now reaches DR21.2 (A), SWR16.1, SWR20.1, SWR7.1
- net LABEL_CR3: now also DR3.2 (A), SWR2.1, DR43.1 (K), DR45.1 (K), SWR24.1; no longer SWL24.1
- net at DR42.2 (A), DR6.2 (A), SWR5.1: now also DR18.1 (K), DR36.1 (K), DR24.1 (K), DR30.1 (K); no longer DL18.1 (K), DL36.1 (K)
- net at SWL12.2: now also DL22.1 (K); no longer DR22.1 (K)
- net at JPR1.1 (A): now also UR4.8 (LPMB); no longer UL4.8 (LPMB)
- net at CL3.1, TL3.1 (Pin_1): now also UL4.3 (TP2)
- net at DL24.1 (K), DL30.1 (K): now also DL18.1 (K), DL36.1 (K), DL42.2 (A), DL6.2 (A), SWL5.1; no longer DR18.1 (K), DR36.1 (K)
- net at RL8.2: now also UL4.16 (TPQ0)
- net at DL5.2 (A), SWL17.1, SWL4.1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: now also DL35.2 (A), SWL13.1; no longer DR35.2 (A), SWR13.1
- net at CR4.1, TR4.1 (Pin_1): now also UR4.4 (TP3); no longer UL4.4 (TP3)
- net at DL30.2 (A): now also QL3.3 (D); no longer QR3.3 (D)
- net at DL8.1 (K): now also SWL1.2
- net at CL6.2, UL2.2 (FB): now also RL6.2, RL7.1; no longer RR6.2, RR7.1
- net at DR12.1 (K): now also SWR5.2
- net at CR6.1, CR8.1, UR2.3 (VOUT)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: now also CR7.1, QR6.3 (D), RR6.1
- net at CR6.2, UR2.2 (FB): now also RR6.2, RR7.1
- net at RL4.1: now also UL2.5 (EN), UL3.1 (Vout); no longer UR2.5 (EN)
- net at DL19.1 (K): now also SWL10.2; no longer SWR10.2
- net at DR2.2 (A), SWR11.1, SWR23.1: now also DR14.2 (A), SWR19.1, SWR1.1, SWR15.1; no longer SWL1.1, SWL15.1
- net at SWL15.2: now also DL26.1 (K)
- net at QR2.3 (D): now also DR24.2 (A); no longer DL24.2 (A)
- net at DR8.1 (K): now also SWR1.2; no longer SWL1.2
- net at SW_BATR1.3 (C): now also JR4.2 (Pin_2)
- net at SWR20.2: now also DR33.1 (K); no longer DL33.1 (K)
- net at SWR4.2: now also DR11.1 (K); no longer DL11.1 (K)
- net at CR2.1, TR2.1 (Pin_1): now also UR4.2 (TP1); no longer UL4.2 (TP1)
- net at SWL4.2: now also DL11.1 (K)
- net at DR26.1 (K): now also SWR15.2
- net at DR40.1 (K): now also SWR25.2; no longer SWL25.2
- net at RL9.2: now also UL4.15 (TPQ1)
- net at SWR13.2: now also DR23.1 (K)
- net at DL12.1 (K): now also SWL5.2; no longer SWR5.2
- net at CR1.1, TR1.1 (Pin_1): now also UR4.1 (TP0); no longer UL4.1 (TP0)
- net at RR9.2: now also UR4.15 (TPQ1); no longer UL4.15 (TPQ1)
- net at RR8.2: now also UR4.16 (TPQ0); no longer UL4.16 (TPQ0)
- net at QL2.3 (D): now also DL24.2 (A)
- removed net BATTERY_RAW+: JL4.1 (Pin_1), LR1.1, RL4.2, UR2.8 (VIN)
- net BATTERY_RAW-: no longer names the net of SW_BATR1.1 (A)
- net BATTERY_RAW-: no longer JL4.2 (Pin_2)
- new net: DR39.1 (K), SWR24.2
- new net: DR43.2 (A), DR44.2 (A), SWR27.1
- new net: QL8.1 (G), RL13.2
- new net: CL5.1, LL1.1, QL8.2 (S), RL2.1, RL4.2, UL2.8 (VIN), UL3.2 (VDD)
- new net: JL4.1 (Pin_1), QL8.3 (D)
- new net: JR3.6 (Pin_6), RR1.2
- new net: DL32.1 (K), SWL19.2
- new net: JR4.1 (Pin_1), QR8.3 (D)
- new net: DR10.1 (K), SWR3.2
- new net: DL13.1 (K), SWL6.2
- new net: DL1.2 (A), DL7.2 (A), SWL10.1, SWL14.1, SWL18.1, SWL22.1, SWL6.1
- new net: DL25.1 (K), SWL14.2
- new net: RR10.2, UR4.14 (TPQ2)
- new net: RR11.2, UR4.13 (TPQ3)
- new net: DR27.1 (K), SWR16.2
- new net: DL9.1 (K), SWL2.2
- new net: DL31.1 (K), SWL18.2
- new net: QR8.1 (G), RR13.1
- new net: DR45.2 (A), DR46.2 (A), SWR28.1
- new net: DR30.2 (A), QR3.3 (D)
- new net: DL37.1 (K), SWL22.2
- new net: DR22.1 (K), SWR12.2
- new net LABEL_CR4: DR28.2 (A), DR4.2 (A), DR44.1 (K), SWR12.1, SWR21.1, SWR25.1, SWR3.1, SWR8.1
Other:
- note added: "1.0V reset"
- note added: "Backflow prevention from USB power"
- note added: "Bluetooth (Arrow1+Arrow2 Combo)"
- note added: "Bluetooth (Arrow1+Arrow3 Combo)"
- note added: "Low VGS(th) required"
- note added: "Reverse connection protection"
- note added: "TOUCH* is active low"
- moved on the sheet: CL1, CL2, CL3, CL4, CL8, CR5, CR6, CR7, DL10, DL11, DL12, DL15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
