File: hardware/dya-dash/right/dya-right.kicad_sch (KiCad schematic)
At the start: 115 parts

Commit message: Finalize v2
Parts:
- added DR43, DR44, DR45, DR46: D, Diode_SMD:D_SOD-123, symbol Device:D
- added QR8: Q_PMOS_GSD, Package_TO_SOT_SMD:SOT-23, symbol Device:Q_PMOS_GSD
- added RR13: 100kΩ, Resistor_SMD:R_0805_2012Metric, symbol Device:R
- added SWR27, SWR28: SW_Push_45deg, 0_dya-kbd:Push_PTS636SM43SMTR, symbol Switch:SW_Push_45deg
- RR15: value 1kΩ -> 100Ω; LCSC C17513 -> C17408
- SW_BATR1: footprint 0_kbd_Parts:TGSW_MSK-12D19 -> 0_dya-kbd:MK-12C02-G015; LCSC (none) -> C2890358
Connections:
- net GNDL: now also RR13.2
- net PINR6: now also SWR27.2, SWR28.2
- net at SW_BATR1.3 (C): now also JR4.2 (Pin_2)
- net LABEL_CR3: now reaches DR21.2 (A), DR3.2 (A), SWR16.1, SWR2.1, SWR20.1, SWR24.1, SWR7.1
- net LABEL_CR3: now also DR43.1 (K), DR45.1 (K)
- net LABEL_CR4: now reaches DR28.2 (A), DR4.2 (A), SWR12.1, SWR21.1, SWR25.1, SWR3.1, SWR8.1
- net LABEL_CR4: now also DR44.1 (K)
- net LABEL_CR5: now reaches DR35.2 (A), DR5.2 (A), SWR13.1, SWR17.1, SWR26.1, SWR4.1, SWR9.1
- net LABEL_CR5: now also DR46.1 (K)
- net BATTERY_RAW+: no longer names the net of CR5.1, LR1.1, RR2.1, RR4.2, UR2.8 (VIN), UR3.2 (VDD)
- net BATTERY_RAW+: now also QR8.2 (S); no longer JR4.1 (Pin_1)
- net BATTERY_RAW-: no longer names the net of SW_BATR1.1 (A)
- net BATTERY_RAW-: no longer JR4.2 (Pin_2)
- new net: DR43.2 (A), DR44.2 (A), SWR27.1
- new net: QR8.1 (G), RR13.1
- new net: DR45.2 (A), DR46.2 (A), SWR28.1
- new net: JR4.1 (Pin_1), QR8.3 (D)
Other:
- note added: "Bluetooth (Arrow1+Arrow2 Combo)"
- note added: "Bluetooth (Arrow1+Arrow3 Combo)"
- note added: "Reverse connection protection"
- moved on the sheet: JR1, JR4, RR2, RR3, SW_BATR1
